File: board/micromouse.sch (KiCad schematic (older format))
At the start: 50 parts, among them J1 Power, J2 SERIAL, J3 PWR_SEL, J4 Front Sense, J5 Left Sense, J6 Right Sense, M1 Left Motor, M2 Right Motor, SW1 SW_SPST, SW2 SW_Push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

Commit message: finished board design
Parts:
- added J7: Back Sense, Connector_PinHeader_2.54mm:PinHeader_1x04_P2.54mm_Vertical, symbol Connector:Conn_01x04_Male
- added MH1, MH2, MH3, MH4, MH5, MH6, MH7, MH8: MountingHole, MountingHole:MountingHole_3.2mm_M3, symbol Mechanical:MountingHole
- added SW5: SW_Push, Button_Switch_THT:SW_PUSH_6mm, symbol Switch:SW_Push
Connections:
- net labels added: BACK_ECHO, BACK_TRIG, BTN1, BTN2
- net labels removed: BTN
- wire segments 231 -> 240
Other:
- moved on the sheet: D1, D2, D3, R12, R13, R14, SW4

Commit message: Finished board layout
Parts:
- added C10, C11: CP, Capacitor_THT:CP_Radial_D5.0mm_P2.50mm, symbol Device:CP
Connections:
- wire segments 240 -> 248
Other:
- moved on the sheet: C9, J2, R1, SW2
Changed lines of the file:
@@
 L Switch:SW_Push SW2
 U 1 1 5B94A6E1
-P 3550 2750
-F 0 "SW2" H 3550 3035 50  0000 C CNN
-F 1 "SW_Push" H 3550 2944 50  0000 C CNN
-F 2 "Button_Switch_THT:SW_PUSH_6mm" H 3550 2950 50  0001 C CNN
-F 3 "" H 3550 2950 50  0001 C CNN
-	1    3550 2750
+P 3950 2750
+F 0 "SW2" H 3950 3035 50  0000 C CNN
+F 1 "SW_Push" H 3950 2944 50  0000 C CNN
+F 2 "Button_Switch_THT:SW_PUSH_6mm" H 3950 2950 50  0001 C CNN
+F 3 "" H 3950 2950 50  0001 C CNN
+	1    3950 2750
 	1    0    0    -1
 $EndComp
@@
 L Device:C C9
 U 1 1 5B94A7E8
-P 3100 2750
-F 0 "C9" H 3215 2796 50  0000 L CNN
-F 1 "0.1uF" H 3215 2705 50  0000 L CNN
-F 2 "Capacitor_SMD:C_0603_1608Metric_Pad1.05x0.95mm_HandSolder" H 3138 2600 50  0001 C CNN
-F 3 "~" H 3100 2750 50  0001 C CNN
-	1    3100 2750
+P 3500 2750
+F 0 "C9" H 3615 2796 50  0000 L CNN
+F 1 "0.1uF" H 3615 2705 50  0000 L CNN
+F 2 "Capacitor_SMD:C_0603_1608Metric_Pad1.05x0.95mm_HandSolder" H 3538 2600 50  0001 C CNN
+F 3 "~" H 3500 2750 50  0001 C CNN
+	1    3500 2750
 	0    1    1    0
 $EndComp
@@
 L Connector:Conn_01x06_Male J2
 U 1 1 5B9C0A8F
-P 2650 2450
-F 0 "J2" H 2756 2828 50  0000 C CNN
-F 1 "SERIAL" H 2756 2737 50  0000 C CNN
-F 2 "Connector_PinHeader_2.54mm:PinHeader_1x06_P2.54mm_Vertical" H 2650 2450 50  0001 C CNN
-F 3 "~" H 2650 2450 50  0001 C CNN
-	1    2650 2450
+P 3050 2450
+F 0 "J2" H 3156 2828 50  0000 C CNN
+F 1 "SERIAL" H 3156 2737 50  0000 C CNN
+F 2 "Connector_PinHeader_2.54mm:PinHeader_1x06_P2.54mm_Vertical" H 3050 2450 50  0001 C CNN
+F 3 "~" H 3050 2450 50  0001 C CNN
+	1    3050 2450
 	1    0    0    -1
 $EndComp
@@
 L power:GND #PWR0121
 U 1 1 5BB5928A
-P 2900 2800
-F 0 "#PWR0121" H 2900 2550 50  0001 C CNN
-F 1 "GND" H 2905 2627 50  0000 C CNN
-F 2 "" H 2900 2800 50  0001 C CNN
-F 3 "" H 2900 2800 50  0001 C CNN
-	1    2900 2800
-	1    0    0    -1
-$EndComp
-Wire Wire Line
-	2900 2800 2900 2350
-Wire Wire Line
-	2900 2350 2850 2350
-Wire Wire Line
-	2900 2350 2900 2250
-Wire Wire Line
-	2900 2250 2850 2250
-Connection ~ 2900 2350
-Wire Wire Line
-	2850 2750 2950 2750
-Text Label 3200 2450 2    50   ~ 0
+P 3300 2800
+F 0 "#PWR0121" H 3300 2550 50  0001 C CNN
+F 1 "GND" H 3305 2627 50  0000 C CNN
+F 2 "" H 3300 2800 50  0001 C CNN
+F 3 "" H 3300 2800 50  0001 C CNN
+	1    3300 2800
+	1    0    0    -1
+$EndComp
+Wire Wire Line
+	3300 2800 3300 2350
+Wire Wire Line
+	3300 2350 3250 2350
+Wire Wire Line
+	3300 2350 3300 2250
+Wire Wire Line
+	3300 2250 3250 2250
+Connection ~ 3300 2350
+Wire Wire Line
+	3250 2750 3350 2750
+Text Label 3600 2450 2    50   ~ 0
 USB_5V
 Wire Wire Line
-	2850 2450 3200 2450
-Text Label 3000 2550 2    50   ~ 0
+	3250 2450 3600 2450
+Text Label 3400 2550 2    50   ~ 0
 RX
-Text Label 3000 2650 2    50   ~ 0
+Text Label 3400 2650 2    50   ~ 0
 TX
 Wire Wire Line
-	3000 2550 2850 2550
-Wire Wire Line
-	2850 2650 3000 2650
+	3400 2550 3250 2550
+Wire Wire Line
+	3250 2650 3400 2650
 $Comp
 L power:+5V #PWR0122
 U 1 1 5BBA84FD
-P 3300 2350
-F 0 "#PWR0122" H 3300 2200 50  0001 C CNN
-F 1 "+5V" H 3315 2523 50  0000 C CNN
-F 2 "" H 3300 2350 50  0001 C CNN
-F 3 "" H 3300 2350 50  0001 C CNN
-	1    3300 2350
+P 3700 2350
+F 0 "#PWR0122" H 3700 2200 50  0001 C CNN
+F 1 "+5V" H 3715 2523 50  0000 C CNN
+F 2 "" H 3700 2350 50  0001 C CNN
+F 3 "" H 3700 2350 50  0001 C CNN
+	1    3700 2350
 	1    0    0    -1
 $EndComp
@@
 L Device:R R1
 U 1 1 5BBA860A
-P 3300 2550
-F 0 "R1" V 3350 2700 50  0000 C CNN
-F 1 "1K" V 3300 2550 50  0000 C CNN
-F 2 "Resistor_SMD:R_0603_1608Metric_Pad1.05x0.95mm_HandSolder" V 3230 2550 50  0001 C CNN
-F 3 "~" H 3300 2550 50  0001 C CNN
-	1    3300 2550
+P 3700 2550
+F 0 "R1" V 3750 2700 50  0000 C CNN
+F 1 "1K" V 3700 2550 50  0000 C CNN
+F 2 "Resistor_SMD:R_0603_1608Metric_Pad1.05x0.95mm_HandSolder" V 3630 2550 50  0001 C CNN
+F 3 "~" H 3700 2550 50  0001 C CNN
+	1    3700 2550
 	-1   0    0    1
 $EndComp
 Wire Wire Line
-	3300 2350 3300 2400
-Wire Wire Line
-	3250 2750 3300 2750
-Wire Wire Line
-	3300 2700 3300 2750
-Connection ~ 3300 2750
-Wire Wire Line
-	3300 2750 3350 2750
+	3700 2350 3700 2400
+Wire Wire Line
+	3650 2750 3700 2750
+Wire Wire Line
+	3700 2700 3700 2750
+Connection ~ 3700 2750
+Wire Wire Line
+	3700 2750 3750 2750
 $Comp
 L power:GND #PWR0123
 U 1 1 5BBC41A7
-P 3800 2800
-F 0 "#PWR0123" H 3800 2550 50  0001 C CNN
-F 1 "GND" H 3805 2627 50  0000 C CNN
-F 2 "" H 3800 2800 50  0001 C CNN
-F 3 "" H 3800 2800 50  0001 C CNN
-	1    3800 2800
-	1    0    0    -1
-$EndComp
-Wire Wire Line
-	3800 2800 3800 2750
-Wire Wire Line
-	3800 2750 3750 2750
-Text Label 3450 2850 2    50   ~ 0
+P 4200 2800
+F 0 "#PWR0123" H 4200 2550 50  0001 C CNN
+F 1 "GND" H 4205 2627 50  0000 C CNN
+F 2 "" H 4200 2800 50  0001 C CNN
+F 3 "" H 4200 2800 50  0001 C CNN
+	1    4200 2800
+	1    0    0    -1
+$EndComp
+Wire Wire Line
+	4200 2800 4200 2750
+Wire Wire Line
+	4200 2750 4150 2750
+Text Label 3850 2850 2    50   ~ 0
 RST
 Wire Wire Line
-	3450 2850 3300 2850
-Wire Wire Line
-	3300 2850 3300 2750
+	3850 2850 3700 2850
+Wire Wire Line
+	3700 2850 3700 2750
 $Comp
 L Connector:Conn_01x03_Male J3
@@
 	3000 4000 3000 3300
 Wire Notes Line
-	700  2000 2350 2000
-Wire Notes Line
-	2350 2000 2350 3000
-Wire Notes Line
-	2350 3000 700  3000
-Wire Notes Line
 	700  3000 700  2000
 Wire Notes Line
-	2600 2000 2600 3050
-Wire Notes Line
-	2600 3050 3900 3050
-Wire Notes Line
-	3900 3050 3900 2000
-Wire Notes Line
-	3900 2000 2600 2000
+	3000 2000 3000 3050
+Wire Notes Line
+	3000 3050 4300 3050
+Wire Notes Line
+	4300 3050 4300 2000
+Wire Notes Line
+	4300 2000 3000 2000
 Wire Notes Line
 	3400 700  3400 1750
@@
 Wire Wire Line
 	6850 5500 6400 5500
+$Comp
+L Device:CP C10
+U 1 1 5BB793BF
+P 2350 2500
+F 0 "C10" H 2400 2400 50  0000 L CNN
+F 1 "CP" H 2400 2600 50  0000 L CNN
+F 2 "Capacitor_THT:CP_Radial_D5.0mm_P2.50mm" H 2388 2350 50  0001 C CNN
+F 3 "~" H 2350 2500 50  0001 C CNN
+	1    2350 2500
+	1    0    0    -1
+$EndComp
+$Comp
+L Device:CP C11
+U 1 1 5BB7946B
+P 2600 2500
+F 0 "C11" H 2650 2400 50  0000 L CNN
+F 1 "CP" H 2650 2600 50  0000 L CNN
+F 2 "Capacitor_THT:CP_Radial_D5.0mm_P2.50mm" H 2638 2350 50  0001 C CNN
+F 3 "~" H 2600 2500 50  0001 C CNN
+	1    2600 2500
+	1    0    0    -1
+$EndComp
+Wire Wire Line
+	2100 2700 2350 2700
+Wire Wire Line
+	2350 2700 2350 2650
+Connection ~ 2100 2700
+Wire Wire Line
+	2350 2700 2600 2700
+Wire Wire Line
+	2600 2700 2600 2650
+Connection ~ 2350 2700
+Wire Wire Line
+	2100 2300 2350 2300
+Wire Wire Line
+	2350 2300 2350 2350
+Connection ~ 2100 2300
+Wire Wire Line
+	2350 2300 2600 2300
+Wire Wire Line
+	2600 2300 2600 2350
+Connection ~ 2350 2300
+Wire Notes Line
+	700  2000 2800 2000
+Wire Notes Line
+	2800 2000 2800 3000
+Wire Notes Line
+	2800 3000 700  3000
+Wire Notes Line
+	4800 4500 4800 6550
+Wire Notes Line
+	4800 6550 6950 6550
+Wire Notes Line
+	6950 6550 6950 4500
+Wire Notes Line
+	6950 4500 4800 4500
 $EndSCHEMATC

Commit message: Finish small board
Parts:
- removed J1: Power, Connector_PinHeader_2.54mm:PinHeader_1x02_P2.54mm_Vertical, symbol Connector:Conn_01x02_Male
- removed SW2: SW_Push, Button_Switch_THT:SW_PUSH_6mm, symbol Switch:SW_Push
- added BT1, BT2: 3x AA, Connector_PinHeader_2.54mm:PinHeader_2x01_P2.54mm_Vertical, symbol Device:Battery
- added J1: PowerBtnLower, Connector_PinSocket_2.54mm:PinSocket_1x05_P2.54mm_Vertical, symbol Connector:Conn_01x05_Male
- added J12: MotorsUpper, Connector_PinSocket_2.54mm:PinSocket_1x05_P2.54mm_Vertical, symbol Connector:Conn_01x05_Female
- added J8: PowerBtnUpper, Connector_PinSocket_2.54mm:PinSocket_1x05_P2.54mm_Vertical, symbol Connector:Conn_01x05_Female
- added J9: MotorsLower, Connector_PinHeader_2.54mm:PinHeader_1x05_P2.54mm_Vertical, symbol Connector:Conn_01x05_Male
- D1, D2, D3: footprint LED_THT:LED_D5.0mm -> LED_THT:LED_D5.0mm_Horizontal_O1.27mm_Z3.0mm
- SW1: footprint Button_Switch_THT:SW_DIP_SPSTx01_Slide_6.7x4.1mm_W7.62mm_P2.54mm_LowProfile -> Connector_PinHeader_2.54mm:PinHeader_2x01_P2.54mm_Vertical
- U2: footprint Package_TO_SOT_THT:TO-220-3_Horizontal_TabDown -> Package_TO_SOT_THT:TO-220-3_Vertical
Connections:
- net labels added: +5VD, BTN1_T, BTN2_T, GNDD, LEFT_DIR_T, LEFT_STEP_T, M_ENABLE_T, RIGHT_DIR_T, RIGHT_STEP_T, USB_5V_T
- wire segments 248 -> 274
Other:
- moved on the sheet: C1, C10, C11, C2, C3, C4, C5, C6, C7, C8, C9, D1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

Commit message: Final 2-board design
Parts:
- D1: footprint LED_THT:LED_D5.0mm_Horizontal_O1.27mm_Z3.0mm -> LED_SMD:LED_0603_1608Metric_Pad1.05x0.95mm_HandSolder
- D2, D3: footprint LED_THT:LED_D5.0mm_Horizontal_O1.27mm_Z3.0mm -> LED_THT:LED_D3.0mm
- U3, U4: symbol drv8825:drv8825 -> micromouse-rescue:drv8825-drv8825
Other:
- moved on the sheet: D1, R12
Changed lines of the file:
@@
 F 0 "D2" H 2500 5500 50  0000 C CNN
 F 1 "LED" H 2250 5500 50  0000 C CNN
-F 2 "LED_THT:LED_D5.0mm_Horizontal_O1.27mm_Z3.0mm" H 2400 5450 50  0001 C CNN
+F 2 "LED_THT:LED_D3.0mm" H 2400 5450 50  0001 C CNN
 F 3 "~" H 2400 5450 50  0001 C CNN
 	1    2400 5450
@@
 $EndComp
 $Comp
-L drv8825:drv8825 U3
+L micromouse-rescue:drv8825-drv8825 U3
 U 1 1 5B99F760
 P 7950 4050
@@
 $EndComp
 $Comp
-L drv8825:drv8825 U4
+L micromouse-rescue:drv8825-drv8825 U4
 U 1 1 5B9BBE80
 P 7950 5600
@@
 F 0 "D3" H 2700 5500 50  0000 C CNN
 F 1 "LED" H 2450 5500 50  0000 C CNN
-F 2 "LED_THT:LED_D5.0mm_Horizontal_O1.27mm_Z3.0mm" H 2600 5450 50  0001 C CNN
+F 2 "LED_THT:LED_D3.0mm" H 2600 5450 50  0001 C CNN
 F 3 "~" H 2600 5450 50  0001 C CNN
 	1    2600 5450
@@
 L Device:R R12
 U 1 1 5BEAF8F4
-P 2200 5800
-F 0 "R12" V 2150 5600 50  0000 L CNN
-F 1 "470" V 2200 5750 50  0000 L CNN
-F 2 "Resistor_SMD:R_0603_1608Metric_Pad1.05x0.95mm_HandSolder" V 2130 5800 50  0001 C CNN
-F 3 "~" H 2200 5800 50  0001 C CNN
-	1    2200 5800
+P 8650 2600
+F 0 "R12" V 8600 2400 50  0000 L CNN
+F 1 "470" V 8650 2550 50  0000 L CNN
+F 2 "Resistor_SMD:R_0603_1608Metric_Pad1.05x0.95mm_HandSolder" V 8580 2600 50  0001 C CNN
+F 3 "~" H 8650 2600 50  0001 C CNN
+	1    8650 2600
 	1    0    0    -1
 $EndComp
@@
 L Device:LED D1
 U 1 1 5BEAF8FA
-P 2200 5450
-F 0 "D1" H 2300 5500 50  0000 C CNN
-F 1 "LED" H 2050 5500 50  0000 C CNN
-F 2 "LED_THT:LED_D5.0mm_Horizontal_O1.27mm_Z3.0mm" H 2200 5450 50  0001 C CNN
-F 3 "~" H 2200 5450 50  0001 C CNN
-	1    2200 5450
+P 8650 2250
+F 0 "D1" H 8750 2300 50  0000 C CNN
+F 1 "LED" H 8500 2300 50  0000 C CNN
+F 2 "LED_SMD:LED_0603_1608Metric_Pad1.05x0.95mm_HandSolder" H 8650 2250 50  0001 C CNN
+F 3 "~" H 8650 2250 50  0001 C CNN
+	1    8650 2250
 	0    -1   -1   0
 $EndComp
 Wire Wire Line
-	2200 5600 2200 5650
-Wire Wire Line
-	2200 5950 2200 6000
-Wire Wire Line
-	2200 5250 2200 5300
-Wire Notes Line
-	2100 6250 2100 5050
+	8650 2400 8650 2450
+Wire Wire Line
+	8650 2750 8650 2800
+Wire Wire Line
+	8650 2050 8650 2100
+Wire Notes Line
+	2250 6250 2250 5050
 Text Notes 6500 1700 0    50   ~ 0
 8.2v min input
@@
 	2750 5050 2750 6250
 Wire Notes Line
-	2100 6250 2750 6250
-Wire Notes Line
-	2100 5050 2750 5050
+	2250 6250 2750 6250
+Wire Notes Line
+	2250 5050 2750 5050
 $Comp
 L Connector:Conn_01x04_Male J7
@@
 	8200 1850 8200 3050
 Wire Notes Line
-	8200 3050 8600 3050
-Wire Notes Line
-	8600 3050 8600 1850
-Wire Notes Line
-	8600 1850 8200 1850
+	8200 3050 8750 3050
+Wire Notes Line
+	8750 3050 8750 1850
+Wire Notes Line
+	8750 1850 8200 1850
 $Comp
 L Connector:Conn_01x05_Male J9
@@
 	5850 1000 5800 1000
 $Comp
-L power:+5VD #PWR0131
+L power:+5V #PWR0131
 U 1 1 5BF1FC61
-P 2200 5250
-F 0 "#PWR0131" H 2200 5100 50  0001 C CNN
-F 1 "+5VD" H 2215 5423 50  0000 C CNN
-F 2 "" H 2200 5250 50  0001 C CNN
-F 3 "" H 2200 5250 50  0001 C CNN
-	1    2200 5250
-	1    0    0    -1
-$EndComp
-$Comp
-L power:GNDD #PWR0132
+P 8650 2050
+F 0 "#PWR0131" H 8650 1900 50  0001 C CNN
+F 1 "+5V" H 8665 2223 50  0000 C CNN
+F 2 "" H 8650 2050 50  0001 C CNN
+F 3 "" H 8650 2050 50  0001 C CNN
+	1    8650 2050
+	1    0    0    -1
+$EndComp
+$Comp
+L power:GND #PWR0132
 U 1 1 5BF1FEF7
-P 2200 6000
-F 0 "#PWR0132" H 2200 5750 50  0001 C CNN
-F 1 "GNDD" H 2204 5845 50  0000 C CNN
-F 2 "" H 2200 6000 50  0001 C CNN
-F 3 "" H 2200 6000 50  0001 C CNN
-	1    2200 6000
+P 8650 2800
+F 0 "#PWR0132" H 8650 2550 50  0001 C CNN
+F 1 "GND" H 8654 2645 50  0000 C CNN
+F 2 "" H 8650 2800 50  0001 C CNN
+F 3 "" H 8650 2800 50  0001 C CNN
+	1    8650 2800
 	1    0    0    -1
 $EndComp
@@
 Wire Wire Line
 	4150 4500 4500 4500
+Entry Wire Line
+	2950 5650 3050 5750
 $EndSCHEMATC
