File: board/board2.sch (KiCad schematic (older format))
At the start: 71 parts, among them J1 Battery, J2 Conn_01x06_Male, J3 Conn_ARM_JTAG_SWD_10, J4 Range_Front, J5 Range_Left, J6 Range_Right, J7 Battery, SW1 RST, SW2 SW_Push, SW3 SW_Push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

Commit message: Board redesign
 - add IMU6500
 - only one battery
 - half the size
 - op amp buffer on battery monitor
 - 4 layer board
 - and more
Parts:
- removed D5: D_Zener, Diode_THT:D_T-1_P2.54mm_Vertical_AnodeUp, symbol Device:D_Zener
- removed H10, H7, H8, H9: MountingHole, MountingHole:MountingHole_2.2mm_M2, symbol Mechanical:MountingHole
- removed J7: Battery, Connector_PinHeader_2.54mm:PinHeader_1x02_P2.54mm_Horizontal, symbol Connector:Conn_01x02_Male
- removed JP1: UART_PWR, Connector_PinHeader_2.54mm:PinHeader_1x02_P2.54mm_Vertical, symbol Device:Jumper_NC_Small
- removed JP2: BOOT0, Connector_PinHeader_2.54mm:PinHeader_1x02_P2.54mm_Vertical, symbol Device:Jumper_NC_Small
- removed JP3: BOOT1, Connector_PinHeader_2.54mm:PinHeader_1x02_P2.54mm_Vertical, symbol Device:Jumper_NC_Small
- removed JP4: BAT_PWR, Connector_PinHeader_2.54mm:PinHeader_1x02_P2.54mm_Vertical, symbol Device:Jumper_NC_Small
- removed JP5: PROG_PWR, Connector_PinHeader_2.54mm:PinHeader_1x02_P2.54mm_Vertical, symbol Device:Jumper_NC_Small
- removed R1, R2: 10K, Resistor_SMD:R_0603_1608Metric, symbol Device:R_Small
- added C17, C18, C19, C20, C21, C22: 0.1uF, Capacitor_SMD:C_0603_1608Metric, symbol Device:C_Small
- added D5: DB2441700L, micromouse_custom:SC-110A-2, symbol Device:D
- added D6: WHITE, LED_SMD:LED_0603_1608Metric, symbol Device:LED
- added JP1: UART_PWR, Connector_PinHeader_2.54mm:PinHeader_1x03_P2.54mm_Vertical_SMD_Pin1Left, symbol Jumper:Jumper_3_Bridged12
- added R1, R12, R2: 10k, Resistor_SMD:R_0603_1608Metric, symbol Device:R
- added R13: 10k, Resistor_SMD:R_0603_1608Metric, symbol Device:R_Small
- added R14, R15, R16, R17, R18, R19: 2.2K, Resistor_SMD:R_0603_1608Metric, symbol Device:R
- added R20: 330, Resistor_SMD:R_0603_1608Metric, symbol Device:R
- added SW5: Power, Connector_PinHeader_2.54mm:PinHeader_2x01_P2.54mm_Vertical_SMD, symbol Switch:SW_SPST
- added TP1: BAT, micromouse_custom:TestPoint_Pad_1.8x1.0mm, symbol Connector:TestPoint
- added TP10, TP11, TP8, TP9: GND, micromouse_custom:TestPoint_Pad_1.8x1.0mm, symbol Connector:TestPoint
- added U6: MCP6001U, Package_TO_SOT_SMD:SOT-23-5, symbol Amplifier_Operational:MCP6001U
- added U7: MPU-6500, Sensor_Motion:InvenSense_QFN-24_4x4mm_P0.5mm, symbol Sensor_Motion:MPU-6500
- C15: footprint Capacitor_THT:CP_Radial_D5.0mm_P2.50mm -> Capacitor_SMD:CP_Elec_4x4.5
- D1: value LED -> RED
- D2: value LED -> GREEN
- D3: value LED -> BLUE
- D4: value LED -> ORANGE
- F1: value 2A -> 1A; footprint Fuse:Fuse_Littelfuse-LVR100 -> micromouse_custom:Littlefuse_154
- H1, H2, H3, H4: value MountingHole -> Corner
- J2: value Conn_01x06_Male -> Serial; footprint Connector_PinHeader_2.54mm:PinHeader_1x06_P2.54mm_Vertical -> Connector_PinHeader_2.54mm:PinHeader_1x08_P2.54mm_Vertical_SMD_Pin1Left; symbol Connector:Conn_01x06_Male -> Connector:Conn_01x08_Male
- J3: value Conn_ARM_JTAG_SWD_10 -> SWD
- J8: renamed from J?; value Conn_02x06_Odd_Even -> Exp; footprint (none) -> Connector_PinHeader_2.00mm:PinHeader_2x06_P2.00mm_Vertical_SMD
- NT1: value Net-Tie_2 -> GND-Tie
- R3: value 2k -> 200k
- R4: value 1k -> 100k
- R5: value 1k -> 10k
- SW1: footprint Button_Switch_THT:SW_PUSH_6mm -> Button_Switch_SMD:SW_SPST_PTS810
- SW2: value SW_Push -> Left; footprint Button_Switch_THT:SW_PUSH_6mm -> Button_Switch_SMD:SW_SPST_PTS810
- SW3: value SW_Push -> Right; footprint Button_Switch_THT:SW_PUSH_6mm -> Button_Switch_SMD:SW_SPST_PTS810
- SW4: value SW_Push -> Center; footprint Button_Switch_THT:SW_PUSH_6mm -> Button_Switch_SMD:SW_SPST_PTS810
- TP2, TP3, TP4, TP5, TP6, TP7: footprint TestPoint:TestPoint_THTPad_D2.5mm_Drill1.2mm -> micromouse_custom:TestPoint_Pad_1.8x1.0mm
- U4: footprint Connector_PinHeader_2.54mm:PinHeader_1x06_P2.54mm_Vertical_SMD_Pin1Left -> Connector_JST:JST_PH_S6B-PH-SM4-TB_1x06-1MP_P2.00mm_Horizontal
- U5: footprint Connector_PinHeader_2.54mm:PinHeader_1x06_P2.54mm_Vertical_SMD_Pin1Right -> Connector_JST:JST_PH_S6B-PH-SM4-TB_1x06-1MP_P2.00mm_Horizontal
Connections:
- net labels added: IMU_INT
- net labels removed: BOOT0, BOOT1, PC7
- wire segments 306 -> 400
- no-connect marks 5 -> 10
Other:
- note added: "Bat Measurement"
- note added: "Buttons & LEDs"
- note added: "Bypass & Bulk"
- note added: "Clock"
- note added: "Debug"
- note added: "EXTI7"
- note added: "Expansion"
- note added: "IMU"
- note added: "Microcontroller"
- note added: "Motors"
- note added: "Mounting Holes"
- note added: "Power Supply"
- note added: "Program"
- note added: "Range Sensors"
- note added: "Test"
- moved on the sheet: C1, C10, C11, C12, C13, C14, C15, C16, C2, C3, C4, C5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

Commit message: Final board layout
Parts:
- removed J8: Exp, Connector_PinHeader_2.00mm:PinHeader_2x06_P2.00mm_Vertical_SMD, symbol Connector_Generic:Conn_02x06_Odd_Even
- removed JP1: UART_PWR, Connector_PinHeader_2.54mm:PinHeader_1x03_P2.54mm_Vertical_SMD_Pin1Left, symbol Jumper:Jumper_3_Bridged12
- added J7: POWER, Connector_PinHeader_2.54mm:PinHeader_1x04_P2.54mm_Vertical_SMD_Pin1Left, symbol Connector:Conn_01x04_Male
- added J8: EXP, Connector_PinHeader_2.00mm:PinHeader_2x07_P2.00mm_Vertical_SMD, symbol Connector_Generic:Conn_02x07_Odd_Even
- U4, U5: footprint Connector_JST:JST_PH_S6B-PH-SM4-TB_1x06-1MP_P2.00mm_Horizontal -> Connector_Molex:Molex_PicoBlade_53261-0671_1x06-1MP_P1.25mm_Horizontal
Connections:
- net +3V3: now also J7.4 (Pin_4), J8.2 (Pin_2)
- net +BATT: now also J7.2 (Pin_2)
- net GNDD: now also J7.1 (Pin_1), J8.1 (Pin_1)
- net PA3: now also J8.11 (Pin_11)
- net PA4: now also J8.12 (Pin_12)
- net PB0: now also J8.10 (Pin_10)
- net PB4: now also J8.14 (Pin_14)
- net PB5: now also J8.13 (Pin_13)
- net PC13: now also J8.7 (Pin_7)
- net PC14: now also J8.9 (Pin_9)
- net PC15: now also J8.5 (Pin_5)
- net PC8: now also J8.6 (Pin_6)
- net PD2: now also J8.8 (Pin_8)
- net R_SCL: now also J8.3 (Pin_3)
- net R_SDA: now also J8.4 (Pin_4)
- net at J2.3 (Pin_3): now also J7.3 (Pin_3)
Changed lines of the file:
@@
 RTS
-$Comp
-L power:GNDD #PWR0126
-U 1 1 5C790694
-P 1200 7750
-F 0 "#PWR0126" H 1200 7500 50  0001 C CNN
-F 1 "GNDD" H 1204 7595 50  0000 C CNN
-F 2 "" H 1200 7750 50  0001 C CNN
-F 3 "" H 1200 7750 50  0001 C CNN
-	1    1200 7750
-	1    0    0    -1
-$EndComp
 $Comp
 L power:+3.3V #PWR0127
 U 1 1 5C7907B0
-P 950 6700
-F 0 "#PWR0127" H 950 6550 50  0001 C CNN
-F 1 "+3.3V" H 965 6873 50  0000 C CNN
-F 2 "" H 950 6700 50  0001 C CNN
-F 3 "" H 950 6700 50  0001 C CNN
-	1    950  6700
+P 950 6750
+F 0 "#PWR0127" H 950 6600 50  0001 C CNN
+F 1 "+3.3V" H 965 6923 50  0000 C CNN
+F 2 "" H 950 6750 50  0001 C CNN
+F 3 "" H 950 6750 50  0001 C CNN
+	1    950  6750
 	1    0    0    -1
 $EndComp
@@
 Wire Wire Line
 	1150 7150 1250 7150
-Wire Wire Line
-	1250 7150 1250 6900
 Wire Wire Line
 	1500 7450 1150 7450
@@
 Text Label 9850 4450 2    50   ~ 0
 PA3
-Text Label 8900 4450 0    50   ~ 0
+Text Label 8950 4450 0    50   ~ 0
 PA4
-Text Label 8900 4350 0    50   ~ 0
+Text Label 8950 4350 0    50   ~ 0
 PB0
-Text Label 8900 4550 0    50   ~ 0
+Text Label 8950 4550 0    50   ~ 0
 PB4
 Text Label 9850 4550 2    50   ~ 0
 PB5
+Text Label 9850 4150 2    50   ~ 0
+PC15
 Text Label 9850 4350 2    50   ~ 0
-PC15
+PC14
 Text Label 9850 4250 2    50   ~ 0
-PC14
-Text Label 9850 4150 2    50   ~ 0
 PC13
-Text Label 8900 4150 0    50   ~ 0
+Text Label 8950 4150 0    50   ~ 0
 PC8
 $Comp
 L power:+3.3V #PWR0131
 U 1 1 5C6FB475
-P 8950 4000
-F 0 "#PWR0131" H 8950 3850 50  0001 C CNN
-F 1 "+3.3V" H 9100 4050 50  0000 C CNN
-F 2 "" H 8950 4000 50  0001 C CNN
-F 3 "" H 8950 4000 50  0001 C CNN
-	1    8950 4000
-	1    0    0    -1
-$EndComp
-Wire Wire Line
-	8950 4000 8950 4050
-Wire Wire Line
-	8950 4050 9150 4050
-Wire Wire Line
-	9150 4150 8900 4150
-Wire Wire Line
-	8900 4250 9150 4250
-Wire Wire Line
-	9150 4350 8900 4350
-Wire Wire Line
-	8900 4450 9150 4450
-Wire Wire Line
-	8900 4550 9150 4550
+P 8950 3900
+F 0 "#PWR0131" H 8950 3750 50  0001 C CNN
+F 1 "+3.3V" H 9050 3900 50  0000 C CNN
+F 2 "" H 8950 3900 50  0001 C CNN
+F 3 "" H 8950 3900 50  0001 C CNN
+	1    8950 3900
+	1    0    0    -1
+$EndComp
+Wire Wire Line
+	8950 3900 8950 3950
+Wire Wire Line
+	8950 3950 9150 3950
+Wire Wire Line
+	9150 4150 8950 4150
+Wire Wire Line
+	8950 4250 9150 4250
+Wire Wire Line
+	9150 4350 8950 4350
+Wire Wire Line
+	8950 4450 9150 4450
+Wire Wire Line
+	8950 4550 9150 4550
 Wire Wire Line
 	9650 4550 9850 4550
@@
 L power:GNDD #PWR0140
 U 1 1 5C8808B8
-P 9950 4100
-F 0 "#PWR0140" H 9950 3850 50  0001 C CNN
-F 1 "GNDD" H 9950 3950 50  0000 C CNN
-F 2 "" H 9950 4100 50  0001 C CNN
-F 3 "" H 9950 4100 50  0001 C CNN
-	1    9950 4100
-	1    0    0    -1
-$EndComp
-Wire Wire Line
-	9950 4100 9950 4050
-Wire Wire Line
-	9950 4050 9650 4050
-$Comp
-L Connector_Generic:Conn_02x06_Odd_Even J8
-U 1 1 5C89C302
-P 9450 4250
-F 0 "J8" H 9600 4550 50  0000 C CNN
-F 1 "Exp" H 9450 4550 50  0000 C CNN
-F 2 "Connector_PinHeader_2.00mm:PinHeader_2x06_P2.00mm_Vertical_SMD" H 9450 4250 50  0001 C CNN
-F 3 "~" H 9450 4250 50  0001 C CNN
-	1    9450 4250
-	-1   0    0    -1
-$EndComp
+P 9950 4000
+F 0 "#PWR0140" H 9950 3750 50  0001 C CNN
+F 1 "GNDD" H 9950 3850 50  0000 C CNN
+F 2 "" H 9950 4000 50  0001 C CNN
+F 3 "" H 9950 4000 50  0001 C CNN
+	1    9950 4000
+	1    0    0    -1
+$EndComp
+Wire Wire Line
+	9950 4000 9950 3950
+Wire Wire Line
+	9950 3950 9650 3950
 Text Notes 5800 6050 0    50   ~ 0
 ADC12_IN9
@@
 Text Notes 3400 6750 0    50   ~ 0
 EXTI7
-Text Label 8900 4250 0    50   ~ 0
+Text Label 8950 4250 0    50   ~ 0
 PD2
-Text Label 1800 6750 2    50   ~ 0
+Text Label 1800 6950 2    50   ~ 0
 BAT_IN
 NoConn ~ 4000 4550
@@
 	1150 7650 1500 7650
 Wire Wire Line
-	1500 6750 1800 6750
-Wire Wire Line
 	1850 1900 1850 1800
 $Comp
@@
 Wire Notes Line
 	7550 4300 6300 4300
-Text Notes 8900 3850 0    50   ~ 0
+Text Notes 9700 3850 0    50   ~ 0
 Expansion
 Wire Notes Line
@@
 F 0 "U5" H 9450 3400 50  0000 L CNN
 F 1 "Right_Motor" V 9900 2900 50  0000 L CNN
-F 2 "Connector_JST:JST_PH_S6B-PH-SM4-TB_1x06-1MP_P2.00mm_Horizontal" H 9750 3100 50  0001 C CNN
+F 2 "Connector_Molex:Molex_PicoBlade_53261-0671_1x06-1MP_P1.25mm_Horizontal" H 9750 3100 50  0001 C CNN
 F 3 "" H 9750 3100 50  0001 C CNN
 	1    9750 3100
@@
 F 0 "U4" H 9450 2500 50  0000 L CNN
 F 1 "Left_Motor" V 9900 2000 50  0000 L CNN
-F 2 "Connector_JST:JST_PH_S6B-PH-SM4-TB_1x06-1MP_P2.00mm_Horizontal" H 9750 2200 50  0001 C CNN
+F 2 "Connector_Molex:Molex_PicoBlade_53261-0671_1x06-1MP_P1.25mm_Horizontal" H 9750 2200 50  0001 C CNN
 F 3 "" H 9750 2200 50  0001 C CNN
 	1    9750 2200
@@
 $EndComp
 Wire Wire Line
-	950  6700 950  6750
-Wire Wire Line
-	950  6750 1000 6750
-$Comp
-L Jumper:Jumper_3_Bridged12 JP1
-U 1 1 5D58B1A7
-P 1250 6750
-F 0 "JP1" H 1250 6954 50  0000 C CNN
-F 1 "UART_PWR" H 1250 6863 50  0000 C CNN
-F 2 "Connector_PinHeader_2.54mm:PinHeader_1x03_P2.54mm_Vertical_SMD_Pin1Left" H 1250 6750 50  0001 C CNN
-F 3 "~" H 1250 6750 50  0001 C CNN
-	1    1250 6750
-	1    0    0    -1
-$EndComp
-$Comp
-L power:GNDD #PWR?
+	950  6750 950  6800
+$Comp
+L power:GNDD #PWR0114
 U 1 1 5CF03D50
 P 2300 4500
-F 0 "#PWR?" H 2300 4250 50  0001 C CNN
+F 0 "#PWR0114" H 2300 4250 50  0001 C CNN
 F 1 "GNDD" H 2304 4345 50  0000 C CNN
 F 2 "" H 2300 4500 50  0001 C CNN
@@
 	1    0    0    -1
 $EndComp
+$Comp
+L Connector:Conn_01x04_Male J7
+U 1 1 5CE1CC1F
+P 1350 6550
+F 0 "J7" V 1412 6694 50  0000 L CNN
+F 1 "POWER" V 1300 6400 50  0000 L CNN
+F 2 "Connector_PinHeader_2.54mm:PinHeader_1x04_P2.54mm_Vertical_SMD_Pin1Left" H 1350 6550 50  0001 C CNN
+F 3 "~" H 1350 6550 50  0001 C CNN
+	1    1350 6550
+	0    1    1    0
+$EndComp
+Wire Wire Line
+	1150 6800 1150 6750
+Wire Wire Line
+	950  6800 1150 6800
+Wire Wire Line
+	1250 6750 1250 7150
+Wire Wire Line
+	1350 6750 1350 6950
+Wire Wire Line
+	1350 6950 1800 6950
+$Comp
+L power:GNDD #PWR0126
+U 1 1 5C790694
+P 1200 7750
+F 0 "#PWR0126" H 1200 7500 50  0001 C CNN
+F 1 "GNDD" H 1204 7595 50  0000 C CNN
+F 2 "" H 1200 7750 50  0001 C CNN
+F 3 "" H 1200 7750 50  0001 C CNN
+	1    1200 7750
+	1    0    0    -1
+$EndComp
+$Comp
+L power:GNDD #PWR0119
+U 1 1 5CF315A5
+P 1450 6850
+F 0 "#PWR0119" H 1450 6600 50  0001 C CNN
+F 1 "GNDD" H 1600 6900 50  0000 C CNN
+F 2 "" H 1450 6850 50  0001 C CNN
+F 3 "" H 1450 6850 50  0001 C CNN
+	1    1450 6850
+	1    0    0    -1
+$EndComp
+Wire Wire Line
+	1450 6750 1450 6850
+$Comp
+L Connector_Generic:Conn_02x07_Odd_Even J8
+U 1 1 5CFBC896
+P 9450 4250
+F 0 "J8" H 9500 4767 50  0000 C CNN
+F 1 "EXP" H 9500 4676 50  0000 C CNN
+F 2 "Connector_PinHeader_2.00mm:PinHeader_2x07_P2.00mm_Vertical_SMD" H 9450 4250 50  0001 C CNN
+F 3 "~" H 9450 4250 50  0001 C CNN
+	1    9450 4250
+	-1   0    0    -1
+$EndComp
+Text Label 8950 4050 0    50   ~ 0
+R_SDA
+Text Label 9850 4050 2    50   ~ 0
+R_SCL
+Wire Wire Line
+	8950 4050 9150 4050
+Wire Wire Line
+	9650 4050 9850 4050
 $EndSCHEMATC

Commit message: board: fix imu footprint
Parts:
- U7: footprint Sensor_Motion:InvenSense_QFN-24_4x4mm_P0.5mm -> Sensor_Motion:InvenSense_QFN-24_3x3mm_P0.4mm
Changed lines of the file:
@@
 F 0 "U7" H 8500 5200 50  0000 C CNN
 F 1 "MPU-6500" H 9200 5200 50  0000 C CNN
-F 2 "Sensor_Motion:InvenSense_QFN-24_4x4mm_P0.5mm" H 8900 4950 50  0001 C CNN
+F 2 "Sensor_Motion:InvenSense_QFN-24_3x3mm_P0.4mm" H 8900 4950 50  0001 C CNN
 F 3 "https://www.mouser.com/datasheet/2/400/MPU-6500-Datasheet2-1112506.pdf" H 8900 5600 50  0001 C CNN
 	1    8900 5750
